File: hardware/UPSMonitorModule/UPSMonitorModule.kicad_pcb (KiCad board)
At the start: 2 copper layers, 100 x 70 mm, 77 parts, among them J1 I2C/ICSP/UART, J10 Screw_Terminal_01x03, J2 Conn_01x06, J3 Conn_01x03, J4 Conn_01x03, J5 Conn_01x02, J6 Conn_01x02, J7 Screw_Terminal_01x03, J8 Screw_Terminal_01x03, J9 Screw_Terminal_01x03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

Commit message: add some new PCB's
Parts:
- removed H1: REMOVE REMOVE REMOVE, esp-map-footprints:ControlModule
