File: hardware/esp32-lora-multi-gateway/psu.kicad_sch (KiCad schematic)
At the start: 31 parts, among them Q1 BC817, Q2 BC817, U5 AMS1117-5.0, U6 LM2596S-3.3, U8 LM2596S-3.3

Commit message: pcb design in progress
Parts:
- D1: footprint Diode_THT:D_DO-27_P5.08mm_Vertical_AnodeUp -> Diode_THT:D_DO-15_P3.81mm_Vertical_AnodeUp
Changed lines of the file:
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@@
 			)
 		)
-		(property "Footprint" "Diode_THT:D_DO-27_P5.08mm_Vertical_AnodeUp"
+		(property "Footprint" "Diode_THT:D_DO-15_P3.81mm_Vertical_AnodeUp"
 			(at 53.34 101.6 0)
 			(effects
