File: hardware/esp32-lora-multi-gateway/esp32-lora-multi-gateway.kicad_pcb (KiCad board)
At the start: 2 copper layers, 140 x 100 mm, 89 parts, among them J1 Conn_01x02, J2 Conn_Coaxial, J3 Conn_Coaxial, J4 Conn_02x03_Counter_Clockwise, J6 Conn_01x06, J7 USB_B, Q1 BC817, Q2 BC817, Q3 BC817, Q4 BC817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

Commit message: add sd card footprint
Parts:
- added J5: Micro_SD_Card_Det1, esp-map-footprints:MicroSD_PUSH-PUSH, F.Cu at (52.4, 79.8)
