File: hardware/esp32-lora-multi-gateway/esp32-lora-multi-gateway.kicad_sch (KiCad schematic)
At the start: 39 parts, among them J2 Conn_Coaxial, J3 Conn_Coaxial, J4 Conn_01x02, J5 ICSP, J6 Conn_01x06, SW1 SW_Push, SW2 SW_Push, U1 lan8720_eth_board, U2 ESP32-WROOM-32, U3 E22-400M30S, U4 E22-900T30S, U5 LM2596S-3.3, U6 AMS1117-5.0, U7 DS1233A-10

Commit message: work on lora gateway
Parts:
- removed C3, C5: 470uF, esp-map-footprints:CAP_10x10_SMD_THT, symbol Device:C_Polarized
- removed C4: 22uF, Capacitor_SMD:C_1812_4532Metric_Pad1.57x3.40mm_HandSolder, symbol Device:C
- removed D1: SS14, Diode_SMD:D_SMA_Handsoldering, symbol Diode:B140-E3
- removed D2: SS14, Diode_SMD:D_SMA_Handsoldering, symbol Diode:1N5822
- removed D3: LED, LED_SMD:LED_1206_3216Metric, symbol Device:LED
- removed J4: Conn_01x02, esp-map-footprints:TerminalBlock-Bornier-2_P5.08mm, symbol Connector_Generic:Conn_01x02
- removed L1: 68uH, esp-map-footprints:L_12x12mm_H8mm, symbol Device:L
- removed R3: 330, Resistor_SMD:R_1206_3216Metric, symbol Device:R
- removed U5: LM2596S-3.3, esp-map-footprints:TO-263-5_TabPin3, symbol Regulator_Switching:LM2596S-3.3
- removed U6: AMS1117-5.0, Package_TO_SOT_SMD:SOT-223-3_TabPin2, symbol Regulator_Linear:AMS1117-5.0
- added BT1: CR2032, esp-map-footprints:BatteryHolder_CR2032, symbol Device:Battery_Cell
- added C10, C13, C8: 100nF, Capacitor_SMD:C_1206_3216Metric_Pad1.33x1.80mm_HandSolder, symbol Device:C
- added C7, C9: 470uF, esp-map-footprints:CAP_10x10_SMD_THT, symbol Device:C_Polarized
- added D9: WS2812B, LED_SMD:LED_WS2812B_PLCC4_5.0x5.0mm_P3.2mm, symbol LED:WS2812B
- added J1: Conn_01x02, esp-map-footprints:TerminalBlock-Bornier-2_P5.08mm, symbol Connector_Generic:Conn_01x02
- added J4: Conn_02x03_Counter_Clockwise, Connector_PinHeader_2.54mm:PinHeader_2x03_P2.54mm_Vertical, symbol Connector_Generic:Conn_02x03_Counter_Clockwise
- added Q3: BC817, Package_TO_SOT_SMD:SOT-23, symbol Transistor_BJT:BC817
- added R18, R19: 10k, Resistor_SMD:R_1206_3216Metric, symbol Device:R
- added U10: PCF8574, Package_SO:SOIC-16W_7.5x10.3mm_P1.27mm, symbol Interface_Expansion:PCF8574
- added U9: DS1307Z+, Package_SO:SOIC-8_3.9x4.9mm_P1.27mm, symbol Timer_RTC:DS1307Z+
- added Y1: 32768Hz, Crystal:Crystal_C38-LF_D3.0mm_L8.0mm_Horizontal_1EP_style1, symbol Device:Crystal_GND3_Small
Connections:
- net +3V3: now also C13.1, J4.2 (Pin_2), U10.16 (VDD), U10.2 (A1)
- net +5V: now also U3.10-VCC, U3.9-VCC, U4.6 (VCC), C10.1, C7.1, C8.1, C9.1, J4.1 (Pin_1); no longer D4.1 (VDD)
- net GND: now also BT1.2 (-), C10.2, C13.2, C7.2, C8.2, C9.2, D9.3 (VSS), J1.1 (Pin_1), J4.4 (Pin_4), Q3.2 (E), U10.1 (A0), U10.3 (A2), U10.8 (VSS), U9.4 (GND), Y1.3
- net INT: now also U10.13 (~{INT})
- net RGBLED: now also R19.1; no longer D4.4 (DIN)
- net SCL: now also U10.14 (SCL), U9.6 (SCL)
- net SDA: now also U10.15 (SDA), U9.5 (SDA)
- net S0_M0: now reaches U4.1 (M0)
- net S0_M0: now also U10.5 (P1)
- net S0_M1: now reaches U4.2 (M1)
- net S0_M1: now also U10.6 (P2)
- net TXD1: now reaches U4.3 (RXD)
- net TXD1: now also U2.29 (IO5)
- net RXD1: now reaches U4.4 (TXD)
- net RXD1: now also U2.26 (IO4)
- net S0_AUX: now reaches U4.5 (AUX)
- net S0_AUX: now also U10.4 (P0)
- net S1_DIO1: now reaches U3.13-DIO1
- net S1_DIO1: now also U10.12 (P7)
- net S1_BUSY: now reaches U3.14-BUSY
- net S1_BUSY: now also U10.9 (P4)
- net S1_NRST: now reaches U3.15-NRESET (15-NRST)
- net S1_NRST: now also U10.10 (P5)
- net S1_MISO: now reaches U3.16-MISO
- net S1_MISO: now also U2.14 (IO12)
- net S1_MOSI: now reaches U3.17-MOSI
- net S1_MOSI: now also U2.16 (IO13)
- net S1_SCK: now reaches U3.18-SCK
- net S1_SCK: now also U2.13 (IO14)
- net S1_CS: now reaches U3.19-NSS
- net S1_CS: now also U2.23 (IO15)
- net S1_RXEN: now reaches U3.6-RXEN
- net S1_RXEN: now also U10.11 (P6)
- net at U3.7-TXEN: now also U3.8-DIO2
- net at D4.2 (DOUT): now also D9.4 (DIN)
- net TXD2: now reaches U2.27 (IO16)
- net TXD2: now also J4.6 (Pin_6)
- net VBAT: now reaches U2.4 (SENSOR_VP)
- net RXD2: now reaches U2.7 (IO35)
- net RXD2: now also J4.5 (Pin_5)
- new net: Q3.1 (B), R19.2
- new net: D4.4 (DIN), Q3.3 (C), R18.2
- new net: U9.1 (X1), Y1.2
- new net: U9.2 (X2), Y1.1
- new net: BT1.1 (+), U9.3 (VBAT)
- new net +5V_AUX: D4.1 (VDD), D9.1 (VDD), R18.1, U9.8 (VCC)
- new net +5V_EN: U10.7 (P3)
- new net Power Supply/Vin: J1.2 (Pin_2)
- no-connect marks 7 -> 8
Other:
- added sheet Power Supply (psu.kicad_sch)
- note added: "-> dev. RX -> dev. TX"
- note added: "EXT. EXPANSION PORT"
- note added: "HSPI: LORA400 MISO: IO12 MOSI: IO13 SCK: IO14 CS: IO15"
- note added: "I/O EXPANDER"
- note added: "I2C ADDR: 0x45 (READ) 0x44(WRITE)"
- note added: "I2C ADDR: 0x68"
- note added: "LORA MODEM <S0>: 900MHz"
- note added: "LORA MODEM <S1>: 433MHz"
- note added: "RTC DS1307Z"
- note added: "UART0: PC U0TX: IO1 U0RX: IO3 UART1: LORA900 U1TX: IO5 U1RX: IO4 UART2: EXT U2TX: IO16 U2RX: IO35"
- note added: "todo-list: -TEST WS2812B DRIVER USING OUT PIN FROM DS1307Z -DEFINE EXT. PINOUT -TEST HSPI -SIMULATE PSU PROTECTIONS -ADD CANBUS PROTOCOL?? -ADD USB PORT & CH340G / FTDI -ADD OVER VOLTAGE PROT. -ADD EXT. HSPI EXPANSION PORT WITH CHIP SELECT -ADD SPI SD CARD SLOT"
- moved on the sheet: C1, C2, D4, J2, J3, J5, U2, U3, U4

Commit message: wip
Parts:
- removed J5: ICSP, Connector_PinSocket_2.54mm:PinSocket_1x06_P2.54mm_Vertical, symbol Connector_Generic:Conn_01x06
- removed R8: 10k, Resistor_SMD:R_1206_3216Metric, symbol Device:R
- removed SW1, SW2: SW_Push, Button_Switch_THT:SW_PUSH_6mm, symbol Switch:SW_Push
- added J5: Micro_SD_Card_Det1, symbol Connector:Micro_SD_Card_Det1
- added R25: 10k, Resistor_SMD:R_1206_3216Metric, symbol Device:R
- R7: Fitted (none) -> Yes
Connections:
- net +3V3: now also J5.4 (VDD), R25.1
- net GND: now also J5.10 (SHIELD), J5.6 (VSS)
- net RESET: now also R25.2; no longer R7.2
- net USB_ON: now reaches U2.5 (SENSOR_VN)
- net S1_MISO renamed HSPI_MISO
- net HSPI_MISO: now also J5.7 (DAT0)
- net S1_MOSI renamed HSPI_MOSI
- net HSPI_MOSI: now also J5.3 (CMD)
- net S1_SCK renamed HSPI_SCK
- net HSPI_SCK: now also J5.5 (CLK)
- new net SD_CS: J5.2 (DAT3/CD)
- new net SD_DET: J5.9 (DET), R7.2
- no-connect marks 8 -> 10
Other:
- added sheet USB-UART (usbuart.kicad_sch)
- note added: "SD CARD"
- note added: "USB-UART PORT"
- note added: "todo-list: -DEFINE EXT. PINOUT -TEST HSPI -ADD EXT. HSPI EXPANSION PORT WITH CHIP SELECT -ADD CANBUS PROTOCOL?? -SIMULATE PSU PROTECTIONS done -ADD USB PORT & CH340G / FTDI done -ADD OVER VOLTAGE PROT. won't do. -ADD SPI SD CARD SLOT done"
- note removed: "PUSHBUTTONS"
- note removed: "UART Connector"
- note removed: "todo-list: -TEST WS2812B DRIVER USING OUT PIN FROM DS1307Z -DEFINE EXT. PINOUT -TEST HSPI -SIMULATE PSU PROTECTIONS -ADD CANBUS PROTOCOL?? -ADD USB PORT & CH340G / FTDI -ADD OVER VOLTAGE PROT. -ADD EXT. HSPI EXPANSION PORT WITH CHIP SELECT -ADD SPI SD CARD SLOT"
- moved on the sheet: BT1, FID1, FID2, FID3, H1, H2, H3, H4, J4, U7, U9, Y1

Commit message: pcb design in progress
Parts:
- removed C10: 100nF, Capacitor_SMD:C_1206_3216Metric_Pad1.33x1.80mm_HandSolder, symbol Device:C
- added H5: MountingHole_Pad, MountingHole:MountingHole_3.5mm_Pad, symbol Mechanical:MountingHole_Pad
Connections:
- net GND: now also H5.1
- net at U9.1 (X1): now also Y1.1; no longer Y1.2
- net at U9.2 (X2): now also Y1.2; no longer Y1.1
Other:
- moved on the sheet: H1, H2, H3, H4

Commit message: add sd card footprint
Parts:
- J5: footprint (none) -> esp-map-footprints:MicroSD_PUSH-PUSH
Changed lines of the file:
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@@
 			)
 		)
-		(property "Footprint" ""
+		(property "Footprint" "esp-map-footprints:MicroSD_PUSH-PUSH"
 			(at 298.45 118.11 0)
 			(effects
@@
 			)
 		)
-		(property "Datasheet" "https://tienda.ityt.com.ar/porta-sd/2696-micro-sd-card-z%C3%B3calo-resorte-push-15x15mm-socket-itytarg.html"
+		(property "Datasheet" "https://ityt.com.ar/datasheets/zocalos/SIM/3020-901-0001-MicroSD_PUSH-PUSH.pdf"
 			(at 246.38 133.35 0)
 			(effects
